File: Custom EMG Sensor/EMG_wristband/EMG_wristband.kicad_sch (KiCad schematic)
At the start: 0 parts

Commit message: KiCad sheet set up and added ADS1299IPAGR in libraries folder for external footprints and symbols.
Other:
- added sheet afe_ads1299 (afe_ads1299.kicad_sch)
- added sheet mcu (mcu.kicad_sch)
- added sheet power (power.kicad_sch)
- added sheet preprocessing (preprocessing.kicad_sch)
- added sheet wifi (wifi.kicad_sch)
Changed lines of the file:
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@@
 	(generator_version "9.0")
 	(paper "A4")
+	(sheet
+		(at 90.17 22.86)
+		(size 53.34 36.83)
+		(exclude_from_sim no)
+		(in_bom yes)
+		(on_board yes)
+		(dnp no)
+		(fields_autoplaced yes)
+		(stroke
+			(width 0.1524)
+			(type solid)
+		)
+		(fill
+			(color 0 0 0 0.0000)
+		)
+		(property "Sheetname" "afe_ads1299"
+			(at 90.17 22.1484 0)
+			(effects
+				(font
+					(size 1.27 1.27)
+				)
+				(justify left bottom)
+			)
+		)
+		(property "Sheetfile" "afe_ads1299.kicad_sch"
+			(at 90.17 60.2746 0)
+			(effects
+				(font
+					(size 1.27 1.27)
+				)
+				(justify left top)
+			)
+		)
+		(instances
+			(project "EMG_wristband"
+				(path "/dcf7d921-9fa7-446a-8676-88c652188ea2"
+					(page "4")
+				)
+			)
+		)
+	)
+	(sheet
+		(at 21.59 123.19)
+		(size 53.34 34.29)
+		(exclude_from_sim no)
+		(in_bom yes)
+		(on_board yes)
+		(dnp no)
+		(fields_autoplaced yes)
+		(stroke
+			(width 0.1524)
+			(type solid)
+		)
+		(fill
+			(color 0 0 0 0.0000)
+		)
+		(property "Sheetname" "preprocessing"
+			(at 21.59 122.4784 0)
+			(effects
+				(font
+					(size 1.27 1.27)
+				)
+				(justify left bottom)
+			)
+		)
+		(property "Sheetfile" "preprocessing.kicad_sch"
+			(at 21.59 158.0646 0)
+			(effects
+				(font
+					(size 1.27 1.27)
+				)
+				(justify left top)
+			)
+		)
+		(instances
+			(project "EMG_wristband"
+				(path "/dcf7d921-9fa7-446a-8676-88c652188ea2"
+					(page "6")
+				)
+			)
+		)
+	)
+	(sheet
+		(at 91.44 72.39)
+		(size 54.61 40.64)
+		(exclude_from_sim no)
+		(in_bom yes)
+		(on_board yes)
+		(dnp no)
+		(fields_autoplaced yes)
+		(stroke
+			(width 0.1524)
+			(type solid)
+		)
+		(fill
+			(color 0 0 0 0.0000)
+		)
+		(property "Sheetname" "wifi"
+			(at 91.44 71.6784 0)
+			(effects
+				(font
+					(size 1.27 1.27)
+				)
+				(justify left bottom)
+			)
+		)
+		(property "Sheetfile" "wifi.kicad_sch"
+			(at 91.44 113.6146 0)
+			(effects
+				(font
+					(size 1.27 1.27)
+				)
+				(justify left top)
+			)
+		)
+		(instances
+			(project "EMG_wristband"
+				(path "/dcf7d921-9fa7-446a-8676-88c652188ea2"
+					(page "5")
+				)
+			)
+		)
+	)
+	(sheet
+		(at 21.59 73.66)
+		(size 52.07 39.37)
+		(exclude_from_sim no)
+		(in_bom yes)
+		(on_board yes)
+		(dnp no)
+		(fields_autoplaced yes)
+		(stroke
+			(width 0.1524)
+			(type solid)
+		)
+		(fill
+			(color 0 0 0 0.0000)
+		)
+		(property "Sheetname" "mcu"
+			(at 21.59 72.9484 0)
+			(effects
+				(font
+					(size 1.27 1.27)
+				)
+				(justify left bottom)
+			)
+		)
+		(property "Sheetfile" "mcu.kicad_sch"
+			(at 21.59 113.6146 0)
+			(effects
+				(font
+					(size 1.27 1.27)
+				)
+				(justify left top)
+			)
+		)
+		(instances
+			(project "EMG_wristband"
+				(path "/dcf7d921-9fa7-446a-8676-88c652188ea2"
+					(page "3")
+				)
+			)
+		)
+	)
+	(sheet
+		(at 20.32 21.59)
+		(size 52.07 38.1)
+		(exclude_from_sim no)
+		(in_bom yes)
+		(on_board yes)
+		(dnp no)
+		(fields_autoplaced yes)
+		(stroke
+			(width 0.1524)
+			(type solid)
+		)
+		(fill
+			(color 0 0 0 0.0000)
+		)
+		(property "Sheetname" "power"
+			(at 20.32 20.8784 0)
+			(effects
+				(font
+					(size 1.27 1.27)
+				)
+				(justify left bottom)
+			)
+		)
+		(property "Sheetfile" "power.kicad_sch"
+			(at 20.32 60.2746 0)
+			(show_name yes)
+			(effects
+				(font
+					(size 1.27 1.27)
+				)
+				(justify left top)
+			)
+		)
+		(instances
+			(project "EMG_wristband"
+				(path "/dcf7d921-9fa7-446a-8676-88c652188ea2"
+					(page "2")
+				)
+			)
+		)
+	)
 	(sheet_instances
 		(path "/"
