File: Custom EMG Sensor/EMG_wristband/mcu.kicad_sch (KiCad schematic)
At the start: 0 parts

Commit message: Added STM32F401RET6 footprint and symbol to project and MCU sheet
Parts:
- added U2: STM32F401RET6, LQFP64-10x10mm, symbol STM32F401RET6:STM32F401RET6
